Commit message: feat: add forward camera and autonomous vision-guided obstacle navigation

File: src/wobble_description/urdf/chassis.xacro (robot description, xacro)
@@ -70,3 +70,45 @@
     <origin xyz="0 0 0.02" rpy="0 0 0"/>
   </joint>
+  <!-- ==================== Forward Vision Camera ==================== -->
+  <link name="camera_link">
+    <!-- Camera Body Housing -->
+    <visual>
+      <origin xyz="0 0 0" rpy="0 0 0"/>
+      <geometry>
+        <box size="0.015 0.025 0.020"/>
+      </geometry>
+      <material name="rubber_black"/>
+    </visual>
+    <!-- Camera Optical Lens Barrel -->
+    <visual>
+      <origin xyz="0.009 0 0" rpy="0 ${pi/2} 0"/>
+      <geometry>
+        <cylinder radius="0.006" length="0.006"/>
+      </geometry>
+      <material name="accent_blue"/>
+    </visual>
+    <collision>
+      <origin xyz="0.004 0 0" rpy="0 0 0"/>
+      <geometry>
+        <box size="0.022 0.025 0.020"/>
+      </geometry>
+    </collision>
+    <inertial>
+      <origin xyz="0 0 0" rpy="0 0 0"/>
+      <mass value="0.015"/>
+      <inertia ixx="1e-6" ixy="0" ixz="0" iyy="1e-6" iyz="0" izz="1e-6"/>
+    </inertial>
+  </link>
+  <joint name="camera_joint" type="fixed">
+    <parent link="base_link"/>
+    <child link="camera_link"/>
+    <origin xyz="${chassis_length/2 + 0.0075} 0 0.0" rpy="0 0 0"/>
+  </joint>
+  <!-- Standard ROS camera optical frame (Z forward, X right, Y down) -->
+  <link name="camera_optical_link"/>
+  <joint name="camera_optical_joint" type="fixed">
+    <parent link="camera_link"/>
+    <child link="camera_optical_link"/>
+    <origin xyz="0.012 0 0" rpy="${-pi/2} 0 ${-pi/2}"/>
+  </joint>
 </robot>

File: src/wobble_description/urdf/gazebo.xacro (robot description, xacro)
@@ -79,3 +79,26 @@
     </sensor>
   </gazebo>
+  <!-- Forward-Facing Autonomous Vision Camera -->
+  <gazebo reference="camera_link">
+    <sensor name="camera" type="camera">
+      <always_on>true</always_on>
+      <update_rate>30</update_rate>
+      <visualize>true</visualize>
+      <topic>/camera/image_raw</topic>
+      <camera_info_topic>/camera/camera_info</camera_info_topic>
+      <camera>
+        <horizontal_fov>1.3962634</horizontal_fov>
+        <image>
+          <width>640</width>
+          <height>480</height>
+          <format>R8G8B8</format>
+        </image>
+        <clip>
+          <near>0.02</near>
+          <far>30.0</far>
+        </clip>
+        <optical_frame_id>camera_optical_link</optical_frame_id>
+      </camera>
+    </sensor>
+  </gazebo>
 </robot>
